File: schematics/DSKY/DSKY_DSP_DCD2_3.sch (KiCad schematic (older format))
At the start: 18 parts, among them U12 74LS20, U36 74LS00, U38 74LS244, U39 74LS244, U42 74LS04, U43 74LS04, U44 74LS04, U46 74LS04, U47 74LS126, U49 74LS154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

Commit message: Add files via upload
Parts:
- renumbered U46 to U42
Changed lines of the file:
@@
 $Comp
 L 74xx:74LS04 U42
-U 3 1 6394A228
+U 1 1 6394A228
 P 1050 3800
 F 0 "U42" H 1050 4117 50  0000 C CNN
@@
 F 2 "" H 1050 3800 50  0001 C CNN
 F 3 "http://www.ti.com/lit/gpn/sn74LS04" H 1050 3800 50  0001 C CNN
-	3    1050 3800
+	1    1050 3800
 	1    0    0    -1
 $EndComp
@@
 	4100 5900 4200 6000
 $Comp
-L 74xx:74LS04 U46
-U 6 1 67822F7A
+L 74xx:74LS04 U42
+U 2 1 67822F7A
 P 3550 6350
-F 0 "U46" H 3650 6600 50  0000 C CNN
+F 0 "U42" H 3650 6600 50  0000 C CNN
 F 1 "74LS04" H 3650 6500 50  0000 C CNN
 F 2 "" H 3550 6350 50  0001 C CNN
 F 3 "http://www.ti.com/lit/gpn/sn74LS04" H 3550 6350 50  0001 C CNN
-	6    3550 6350
+	2    3550 6350
 	1    0    0    -1
 $EndComp
@@
 $EndComp
 $Comp
-L 74xx:74LS04 U46
-U 1 1 6698A908
+L 74xx:74LS04 U42
+U 4 1 6698A908
 P 5450 2700
-F 0 "U46" H 5450 3017 50  0000 C CNN
+F 0 "U42" H 5450 3017 50  0000 C CNN
 F 1 "74LS04" H 5450 2926 50  0000 C CNN
 F 2 "" H 5450 2700 50  0001 C CNN
 F 3 "http://www.ti.com/lit/gpn/sn74LS04" H 5450 2700 50  0001 C CNN
-	1    5450 2700
+	4    5450 2700
 	1    0    0    -1
 $EndComp
@@
 $Comp
 L 74xx:74LS04 U42
-U 6 1 669182D9
+U 3 1 669182D9
 P 5450 1900
 F 0 "U42" H 5450 2217 50  0000 C CNN
@@
 F 2 "" H 5450 1900 50  0001 C CNN
 F 3 "http://www.ti.com/lit/gpn/sn74LS04" H 5450 1900 50  0001 C CNN
-	6    5450 1900
-	1    0    0    -1
-$EndComp
+	3    5450 1900
+	1    0    0    -1
+$EndComp

Commit message: Minor tweaks to the display decoding logic.
Parts:
- removed U12, U69: 74LS20, symbol 74xx:74LS20
- removed U36: 74LS00, symbol 74xx:74LS00
- removed U39: 74LS244, symbol 74xx:74LS244
- removed unit 4 of U47
- removed U67: 74LS10, symbol 74xx:74LS10
- added unit 1 of U47
- added unit 2 of U47
- renumbered U66 to U63
Connections:
- net labels added: ID2[0..3], ID3[0..3], MODE1, MODE2, MODE3, RWD[1..12]
- net labels removed: ID24, ID2[0..4], ID2[4..4], ID34, ID3[0..4], ID3[4..4], OW11, OW[11..11], RWD[0..12]
- wire segments 196 -> 150
- no-connect marks 11 -> 7
Other:
- moved on the sheet: U42D

Commit message: Simplified...
Parts:
- removed U38, U50: 74LS244, symbol 74xx:74LS244
- removed U42, U43, U44: 74LS04, symbol 74xx:74LS04
- added U43: 74LS00, symbol 74xx:74LS00
Connections:
- net labels removed: BI1, BI2, BI3, BI4, BI5, BI6, BI7, BI8, BI[1..8], ID20, ID21, ID22, ID23, ID2[0..3], ID30, ID31, ID32, ID33, ID3[0..3]
- wire segments 150 -> 104
- no-connect marks 7 -> 3
Other:
- note removed: "Display\nHigh"
- note removed: "Display\nLow"
- moved on the sheet: U47A, U47B, U47C, U49

Commit message: Minor tweaks.
Parts:
- added U42: 74LS04, symbol 74xx:74LS04
Connections:
- wire segments 104 -> 105
Other:
- moved on the sheet: U43A
Changed lines of the file:
@@
 	1    0    0    -1
 $EndComp
-Text HLabel 5300 1800 0    50   Input ~ 0
+Text HLabel 5350 1800 0    50   Input ~ 0
 CLK2
 $Comp
 L 74xx:74LS00 U43
 U 1 1 62AB580C
-P 5600 1700
-F 0 "U43" H 5600 2025 50  0000 C CNN
-F 1 "74LS00" H 5600 1934 50  0000 C CNN
-F 2 "" H 5600 1700 50  0001 C CNN
-F 3 "http://www.ti.com/lit/gpn/sn74ls00" H 5600 1700 50  0001 C CNN
-	1    5600 1700
+P 5650 1700
+F 0 "U43" H 5650 2025 50  0000 C CNN
+F 1 "74LS00" H 5650 1934 50  0000 C CNN
+F 2 "" H 5650 1700 50  0001 C CNN
+F 3 "http://www.ti.com/lit/gpn/sn74ls00" H 5650 1700 50  0001 C CNN
+	1    5650 1700
 	1    0    0    -1
 $EndComp
-Text HLabel 5900 1700 2    50   Output ~ 0
+Text HLabel 5950 1700 2    50   Output ~ 0
 WRITE3
 Wire Wire Line
-	5150 1600 5300 1600
+	5150 1600 5350 1600
 Wire Wire Line
 	5150 2450 5350 2450
@@
 Wire Wire Line
 	5500 4400 5800 4400
+$Comp
+L 74xx:74LS04 U42
+U 3 1 6368531B
+P 5650 3100
+F 0 "U42" H 5700 3400 50  0000 C CNN
+F 1 "74LS04" H 5700 3300 50  0000 C CNN
+F 2 "" H 5650 3100 50  0001 C CNN
+F 3 "http://www.ti.com/lit/gpn/sn74LS04" H 5650 3100 50  0001 C CNN
+	3    5650 3100
+	1    0    0    -1
+$EndComp
 Wire Wire Line
-	4300 3100 6550 3100
+	5950 3100 6550 3100
+Wire Wire Line
+	4300 3100 5350 3100
 Wire Bus Line
 	5900 4350 5900 4700

Commit message: Sign processing overhauled.
Parts:
- added U5: 74LS04, symbol 74xx:74LS04
Connections:
- wire segments 105 -> 106
Changed lines of the file:
@@
 $Descr A 11000 8500
 encoding utf-8
-Sheet 6 10
+Sheet 7 11
 Title ""
 Date ""
@@
 NoConn ~ 3150 4700
 NoConn ~ 3150 4600
-Text HLabel 2150 3800 0    50   Input ~ 0
+Text HLabel 1350 3800 0    50   Input ~ 0
 DISP
 $Comp
@@
 Wire Wire Line
 	4300 3100 5350 3100
+$Comp
+L 74xx:74LS04 U5
+U 3 1 61B750FA
+P 1650 3800
+F 0 "U5" H 1650 4117 50  0000 C CNN
+F 1 "74LS04" H 1650 4026 50  0000 C CNN
+F 2 "" H 1650 3800 50  0001 C CNN
+F 3 "http://www.ti.com/lit/gpn/sn74LS04" H 1650 3800 50  0001 C CNN
+	3    1650 3800
+	1    0    0    -1
+$EndComp
+Wire Wire Line
+	1950 3800 2150 3800
 Wire Bus Line
 	5900 4350 5900 4700

Commit message: Overhauled the handling of the sign characters.
Parts:
- removed U5: 74LS04, symbol 74xx:74LS04
Connections:
- wire segments 106 -> 105
Changed lines of the file:
@@
 NoConn ~ 3150 4700
 NoConn ~ 3150 4600
-Text HLabel 1350 3800 0    50   Input ~ 0
+Text HLabel 2150 3800 0    50   Input ~ 0
 DISP
 $Comp
@@
 Wire Wire Line
 	4300 3100 5350 3100
-$Comp
-L 74xx:74LS04 U5
-U 3 1 61B750FA
-P 1650 3800
-F 0 "U5" H 1650 4117 50  0000 C CNN
-F 1 "74LS04" H 1650 4026 50  0000 C CNN
-F 2 "" H 1650 3800 50  0001 C CNN
-F 3 "http://www.ti.com/lit/gpn/sn74LS04" H 1650 3800 50  0001 C CNN
-	3    1650 3800
-	1    0    0    -1
-$EndComp
-Wire Wire Line
-	1950 3800 2150 3800
 Wire Bus Line
 	5900 4350 5900 4700

Commit message: Minor tweaks during implementation.
Parts:
- removed U58, U59: 74LS30, symbol 74xx:74LS30
- added U58: 74LS08, symbol 74xx:74LS08
- added U59: 74LS11, symbol 74xx:74LS11
Connections:
- wire segments 105 -> 97
Other:
- moved on the sheet: U43A, U43B, U47A, U47B, U47C

Commit message: Final tweaks, the DSKY is now complete!
Parts:
- removed U56, U57, U63: 74LS20, symbol 74xx:74LS20
- removed U59: 74LS11, symbol 74xx:74LS11
- added U13: 74LS02, symbol 74xx:74LS02
- added U19: 74LS04, symbol 74xx:74LS04
- added U48, U56, U57: 74LS00, symbol 74xx:74LS00
- added unit 4 of U58
- added U59, U63: 74LS32, symbol 74xx:74LS32
- added U8: 74LS10, symbol 74xx:74LS10
- renumbered U43 to U18
Connections:
- net labels added: CLK3, COMB-A, COMB-B, COMB-C, INDC
- net labels removed: CLK2
- wire segments 97 -> 126
Other:
- moved on the sheet: U18A, U42C, U47A, U47B, U47C, U49, U58C
