File: schematics/DSKY/DSKY_DSP_DCC.sch (KiCad schematic (older format))
At the start: 15 parts, among them U23 74LS138, U24 74LS138, U25 74LS138, U26 74LS138, U27 74LS148, U28 74LS148, U29 74LS138, U30 74LS138, U31 74LS138, U32 74LS138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

Commit message: Minor tweaks to the display decoding logic.
Connections:
- net +5V: no longer U28.10 (IO), U34.10 (IO)
- net L0: now reaches U24.10 (O5)
- net L0: now also U28.10 (IO)
- net H0: now reaches U30.10 (O5)
- net H0: now also U34.10 (IO)
- no-connect marks 50 -> 48
Changed lines of the file:
@@
 NoConn ~ 2300 3500
 NoConn ~ 2300 3400
-NoConn ~ 2300 3300
 NoConn ~ 2300 3200
 NoConn ~ 2300 3000
@@
 Text Label 2750 5100 0    50   ~ 0
 L7
-$Comp
-L power:+5V #PWR0151
-U 1 1 637E2B4B
-P 3000 4400
-F 0 "#PWR0151" H 3000 4250 50  0001 C CNN
-F 1 "+5V" H 3015 4573 50  0000 C CNN
-F 2 "" H 3000 4400 50  0001 C CNN
-F 3 "" H 3000 4400 50  0001 C CNN
-	1    3000 4400
-	1    0    0    -1
-$EndComp
 Wire Wire Line
 	3000 3100 2900 3100
@@
 NoConn ~ 7350 3600
 NoConn ~ 7350 3500
-NoConn ~ 7350 3400
 NoConn ~ 7350 3300
 NoConn ~ 7350 3100
@@
 Text Label 7800 5200 0    50   ~ 0
 H7
-$Comp
-L power:+5V #PWR0170
-U 1 1 638E459E
-P 8050 4500
-F 0 "#PWR0170" H 8050 4350 50  0001 C CNN
-F 1 "+5V" H 8065 4673 50  0000 C CNN
-F 2 "" H 8050 4500 50  0001 C CNN
-F 3 "" H 8050 4500 50  0001 C CNN
-	1    8050 4500
-	1    0    0    -1
-$EndComp
 Wire Wire Line
 	8050 3200 7950 3200
@@
 Text Notes 6450 7150 0    100  ~ 0
 DSKY-DSP-DCC:  Decode High/Low Word\nCopyright 2021, William Glasford
+Wire Wire Line
+	2300 3300 2550 3300
+Entry Wire Line
+	2550 3300 2650 3400
+Text Label 2550 3300 2    50   ~ 0
+L0
+Wire Wire Line
+	3000 4400 2750 4400
+Entry Wire Line
+	2650 4500 2750 4400
+Text Label 2750 4400 0    50   ~ 0
+L0
+Wire Wire Line
+	7350 3400 7600 3400
+Entry Wire Line
+	7600 3400 7700 3500
+Text Label 7600 3400 2    50   ~ 0
+H0
+Wire Wire Line
+	8050 4500 7800 4500
+Entry Wire Line
+	7700 4600 7800 4500
+Text Label 7800 4500 0    50   ~ 0
+H0
 Wire Bus Line
 	6450 6050 6450 6650

Commit message: Simplified...
Connections:
- net BI1 renamed ID30
- net BI2 renamed ID31
- net BI3 renamed ID32
- net BI4 renamed ID33
- net BI5 renamed ID20
- net BI6 renamed ID21
- net BI7 renamed ID22
- net BI8 renamed ID23
Changed lines of the file:
@@
 	5300 4800 5400 4900
 Text HLabel 5450 2850 2    50   Output ~ 0
-BI[1..4]
+ID3[0..3]
 Text HLabel 10450 2950 1    50   Output ~ 0
-BI[5..8]
+ID2[0..3]
 Text Label 5300 4800 2    50   ~ 0
-BI1
+ID30
 Text Label 5300 4150 2    50   ~ 0
-BI2
+ID31
 Text Label 5300 3550 2    50   ~ 0
-BI3
+ID32
 Text Label 5300 3100 2    50   ~ 0
-BI4
+ID33
 Text Label 10350 4900 2    50   ~ 0
-BI5
+ID20
 Text Label 10350 4250 2    50   ~ 0
-BI6
+ID21
 Text Label 10350 3650 2    50   ~ 0
-BI7
+ID22
 Text Label 10350 3200 2    50   ~ 0
-BI8
+ID23
 Text Notes 6450 7150 0    100  ~ 0
 DSKY-DSP-DCC:  Decode High/Low Word\nCopyright 2021, William Glasford

Commit message: DSKY Redesign
Connections:
- net ID20 renamed BCD5
- net ID21 renamed BCD6
- net ID22 renamed BCD7
- net ID23 renamed BCD8
- net ID30 renamed BCD1
- net ID31 renamed BCD2
- net ID32 renamed BCD3
- net ID33 renamed BCD4
Other:
- moved on the sheet: U23, U24, U25, U26, U27, U28, U29, U30, U31, U32, U33, U34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
