File: schematics/DSKY/DSKY_DSP_LCD.sch (KiCad schematic (older format))
At the start: 15 parts, among them U53 ICM7228C, U54 ICM7228C, U55 ICM7228C

Commit message: Add files via upload
Connections:
- net labels removed: MODE1
- wire segments 292 -> 288
- no-connect marks 0 -> 4
Changed lines of the file:
@@
 Text HLabel 1250 1400 0    50   Input ~ 0
 ID1[0..4]
-Wire Wire Line
-	1650 3450 1200 3450
-Wire Wire Line
-	1650 5900 1200 5900
 Text HLabel 1650 900  0    50   Input ~ 0
 WRITE1
@@
 Text HLabel 900  7050 0    50   Input ~ 0
 DA3[1..3]
-$Comp
-L power:+5V #PWR0178
-U 1 1 662FBB7A
-P 1200 5700
-F 0 "#PWR0178" H 1200 5550 50  0001 C CNN
-F 1 "+5V" H 1215 5873 50  0000 C CNN
-F 2 "" H 1200 5700 50  0001 C CNN
-F 3 "" H 1200 5700 50  0001 C CNN
-	1    1200 5700
-	1    0    0    -1
-$EndComp
-Wire Wire Line
-	1200 5900 1200 5700
-$Comp
-L power:+5V #PWR0179
-U 1 1 662FB6B2
-P 1200 3300
-F 0 "#PWR0179" H 1200 3150 50  0001 C CNN
-F 1 "+5V" H 1215 3473 50  0000 C CNN
-F 2 "" H 1200 3300 50  0001 C CNN
-F 3 "" H 1200 3300 50  0001 C CNN
-	1    1200 3300
-	1    0    0    -1
-$EndComp
-Wire Wire Line
-	1200 3450 1200 3300
 Text Notes 1050 1800 2    80   ~ 0
 Decoder1
@@
 Text Notes 1050 6700 2    80   ~ 0
 Decoder3
-Text HLabel 1650 1000 0    50   Input ~ 0
-MODE1
 Text Label 1050 2500 0    50   ~ 0
 DA13
@@
 Text Notes 6350 7200 0    100  ~ 0
 DSKY-DSP-LCD:  LCD Decode Logic\nCopyright 2021, William Glasford
+NoConn ~ 1650 1000
+NoConn ~ 1650 3450
+NoConn ~ 1650 5900
+NoConn ~ 3400 3300
 Wire Bus Line
 	950  7050 950  7600

Commit message: Minor tweaks to the display decoding logic.
Connections:
- net labels added: ID2[0..3], ID3[0..3], MODE1, MODE2, MODE3
- net labels removed: ID24, ID2[0..4], ID34, ID3[0..4]
- wire segments 288 -> 286
- no-connect marks 4 -> 3
Changed lines of the file:
@@
 DP-3
 Text Label 3000 950  0    50   ~ 0
-A-2
+A-1
 Text Label 3000 1050 0    50   ~ 0
-B-2
+B-1
 Text Label 3000 1150 0    50   ~ 0
-C-2
+C-1
 Text Label 3000 1250 0    50   ~ 0
-D-2
+D-1
 Text Label 3000 1350 0    50   ~ 0
-E-2
+E-1
 Text Label 3000 1450 0    50   ~ 0
-F-2
+F-1
 Text Label 3000 1550 0    50   ~ 0
-G-2
+G-1
 Text Label 3000 1650 0    50   ~ 0
-DP-2
+DP-1
 Text Label 5400 950  0    50   ~ 0
 A-2
@@
 A-3
 Text Label 8000 5350 0    50   ~ 0
-A-1
+A-2
 Text Label 8000 2550 0    50   ~ 0
 B-2
@@
 B-3
 Text Label 8000 5450 0    50   ~ 0
-B-1
+B-2
 Text Label 8000 2650 0    50   ~ 0
 C-2
@@
 C-3
 Text Label 8000 5550 0    50   ~ 0
-C-1
+C-2
 Text Label 8000 2750 0    50   ~ 0
 D-2
@@
 D-3
 Text Label 8000 5650 0    50   ~ 0
-D-1
+D-2
 Text Label 8000 2850 0    50   ~ 0
 E-2
@@
 E-3
 Text Label 8000 5750 0    50   ~ 0
-E-1
+E-2
 Text Label 8000 2950 0    50   ~ 0
 F-2
@@
 F-3
 Text Label 8000 5850 0    50   ~ 0
-F-1
+F-2
 Text Label 8000 3050 0    50   ~ 0
 G-2
@@
 G-3
 Text Label 8000 5950 0    50   ~ 0
-G-1
+G-2
 Text Label 8000 3150 0    50   ~ 0
 DP-2
@@
 DP-3
 Text Label 8000 6050 0    50   ~ 0
-DP-1
+DP-2
 Wire Wire Line
 	1650 1550 1400 1550
@@
 Wire Wire Line
 	1650 1950 1400 1950
-Wire Wire Line
-	1650 4400 1400 4400
-Wire Wire Line
-	1650 6850 1400 6850
 Entry Wire Line
 	1300 1650 1400 1550
@@
 	1300 4400 1400 4300
 Entry Wire Line
-	1300 4500 1400 4400
-Entry Wire Line
 	950  4850 1050 4750
 Entry Wire Line
@@
 Entry Wire Line
 	1300 6850 1400 6750
-Entry Wire Line
-	1300 6950 1400 6850
 Entry Wire Line
 	950  7300 1050 7200
@@
 Text Label 1400 6750 0    50   ~ 0
 ID33
-Text Label 1400 4400 0    50   ~ 0
-ID24
-Text Label 1400 6850 0    50   ~ 0
-ID34
 Wire Bus Line
 	1300 1400 1250 1400
@@
 	1300 3900 1250 3900
 Text HLabel 1250 3900 0    50   Input ~ 0
-ID2[0..4]
+ID2[0..3]
 Wire Bus Line
 	1300 6350 1250 6350
 Text HLabel 1250 6350 0    50   Input ~ 0
-ID3[0..4]
+ID3[0..3]
 Wire Bus Line
 	950  4650 900  4650
@@
 Text Notes 6350 7200 0    100  ~ 0
 DSKY-DSP-LCD:  LCD Decode Logic\nCopyright 2021, William Glasford
-NoConn ~ 1650 1000
-NoConn ~ 1650 3450
-NoConn ~ 1650 5900
+NoConn ~ 1650 4400
 NoConn ~ 3400 3300
+NoConn ~ 1650 6850
 Wire Bus Line
 	950  7050 950  7600
@@
 	950  2150 950  2700
 Wire Bus Line
+	1300 3900 1300 4450
+Wire Bus Line
+	1300 6350 1300 6900
+Wire Bus Line
 	1300 1400 1300 2150
 Wire Bus Line
-	1300 3900 1300 4550
-Wire Bus Line
-	1300 6350 1300 7000
-Wire Bus Line
 	7900 650  7900 6350
 Wire Bus Line
@@
 Wire Bus Line
 	2900 600  2900 7650
+Text HLabel 1650 1000 0    50   Input ~ 0
+MODE1
+Text HLabel 1650 3450 0    50   Input ~ 0
+MODE2
+Text HLabel 1650 5900 0    50   Input ~ 0
+MODE3
 $EndSCHEMATC

Commit message: Minor tweaks.
Connections:
- net labels removed: DP-2, DP-3
- wire segments 286 -> 263
- no-connect marks 3 -> 25
Changed lines of the file:
@@
 	2800 6400 2900 6500
 Entry Wire Line
-	2800 6500 2900 6600
-Entry Wire Line
 	2800 6700 2900 6800
 Entry Wire Line
@@
 Entry Wire Line
 	2800 4250 2900 4350
-Entry Wire Line
-	2800 4050 2900 4150
 Entry Wire Line
 	2800 3950 2900 4050
@@
 	2450 6400 2800 6400
 Wire Wire Line
-	2450 6500 2800 6500
-Wire Wire Line
 	2450 6700 2800 6700
 Wire Wire Line
@@
 	2450 3950 2800 3950
 Wire Wire Line
-	2450 4050 2800 4050
-Wire Wire Line
 	2450 3750 2800 3750
 Wire Wire Line
@@
 	3500 1550 3000 1550
 Wire Wire Line
-	3500 1650 3000 1650
-Wire Wire Line
 	3500 2450 3000 2450
 Wire Wire Line
@@
 	5950 1550 5400 1550
 Wire Wire Line
-	5950 1650 5400 1650
-Wire Wire Line
 	5950 2450 5400 2450
 Wire Wire Line
@@
 	5950 3050 5400 3050
 Wire Wire Line
-	5950 3150 5400 3150
-Wire Wire Line
 	5950 3900 5400 3900
 Wire Wire Line
@@
 	5950 4500 5400 4500
 Wire Wire Line
-	5950 4600 5400 4600
-Wire Wire Line
 	5950 5350 5400 5350
 Wire Wire Line
@@
 	5950 5950 5400 5950
 Wire Wire Line
-	5950 6050 5400 6050
-Wire Wire Line
 	8650 1150 8000 1150
 Wire Wire Line
@@
 	8650 1550 8000 1550
 Wire Wire Line
-	8650 1650 8000 1650
-Wire Wire Line
 	8650 2450 8000 2450
 Wire Wire Line
@@
 	8650 3050 8000 3050
 Wire Wire Line
-	8650 3150 8000 3150
-Wire Wire Line
 	8650 3900 8000 3900
 Wire Wire Line
@@
 	8650 4500 8000 4500
 Wire Wire Line
-	8650 4600 8000 4600
-Wire Wire Line
 	8650 5350 8000 5350
 Wire Wire Line
@@
 	8650 5950 8000 5950
 Wire Wire Line
-	8650 6050 8000 6050
-Wire Wire Line
 	9850 950  10400 950
 Wire Wire Line
@@
 	4700 1550 5200 1550
 Wire Wire Line
-	4700 1650 5200 1650
-Wire Wire Line
 	4700 2450 5200 2450
 Wire Wire Line
@@
 	4700 3050 5200 3050
 Wire Wire Line
-	4700 3150 5200 3150
-Wire Wire Line
 	4700 3900 5200 3900
 Wire Wire Line
@@
 	4700 4500 5200 4500
 Wire Wire Line
-	4700 4600 5200 4600
-Wire Wire Line
 	4700 5350 5200 5350
 Wire Wire Line
@@
 	4700 5950 5200 5950
 Wire Wire Line
-	4700 6050 5200 6050
-Wire Wire Line
 	7150 1150 7800 1150
 Wire Wire Line
@@
 	7150 1550 7800 1550
 Wire Wire Line
-	7150 1650 7800 1650
-Wire Wire Line
 	7150 2450 7800 2450
 Wire Wire Line
@@
 	7150 3050 7800 3050
 Wire Wire Line
-	7150 3150 7800 3150
-Wire Wire Line
 	7150 3900 7800 3900
 Wire Wire Line
@@
 	7150 4500 7800 4500
 Wire Wire Line
-	7150 4600 7800 4600
-Wire Wire Line
 	7150 5350 7800 5350
 Wire Wire Line
@@
 	7150 5950 7800 5950
 Wire Wire Line
-	7150 6050 7800 6050
-Wire Wire Line
 	9850 1150 10400 1150
 Wire Wire Line
@@
 	9850 1550 10400 1550
 Wire Wire Line
-	9850 1650 10400 1650
-Wire Wire Line
 	9850 2450 10400 2450
 Wire Wire Line
@@
 	9850 3050 10400 3050
 Wire Wire Line
-	9850 3150 10400 3150
-Wire Wire Line
 	9850 3900 10400 3900
 Wire Wire Line
@@
 	9850 4500 10400 4500
 Wire Wire Line
-	9850 4600 10400 4600
-Wire Wire Line
 	9850 5350 10400 5350
 Wire Wire Line
@@
 Wire Wire Line
 	9850 5950 10400 5950
-Wire Wire Line
-	9850 6050 10400 6050
 Wire Wire Line
 	3500 1750 3000 1750
@@
 	2900 2550 3000 2450
 Entry Wire Line
-	2900 1750 3000 1650
-Entry Wire Line
 	2900 1650 3000 1550
 Entry Wire Line
@@
 	5300 1650 5400 1550
 Entry Wire Line
-	5300 1750 5400 1650
-Entry Wire Line
 	5300 2550 5400 2450
 Entry Wire Line
@@
 	5300 3150 5400 3050
 Entry Wire Line
-	5300 3250 5400 3150
-Entry Wire Line
 	5300 4000 5400 3900
 Entry Wire Line
@@
 	5300 4600 5400 4500
 Entry Wire Line
-	5300 4700 5400 4600
-Entry Wire Line
 	5300 5450 5400 5350
 Entry Wire Line
@@
 	5300 6050 5400 5950
 Entry Wire Line
-	5300 6150 5400 6050
-Entry Wire Line
-	7900 6150 8000 6050
-Entry Wire Line
 	7900 6050 8000 5950
 Entry Wire Line
@@
 	7900 5450 8000 5350
 Entry Wire Line
-	7900 4700 8000 4600
-Entry Wire Line
 	7900 4600 8000 4500
 Entry Wire Line
@@
 	7900 4000 8000 3900
 Entry Wire Line
-	7900 3250 8000 3150
-Entry Wire Line
 	7900 3150 8000 3050
 Entry Wire Line
@@
 	7900 2550 8000 2450
 Entry Wire Line
-	7900 1750 8000 1650
-Entry Wire Line
 	7900 1650 8000 1550
 Entry Wire Line
@@
 	10400 1550 10500 1650
 Entry Wire Line
-	10400 1650 10500 1750
-Entry Wire Line
 	10400 2450 10500 2550
 Entry Wire Line
@@
 	10400 3050 10500 3150
 Entry Wire Line
-	10400 3150 10500 3250
-Entry Wire Line
 	10400 3900 10500 4000
 Entry Wire Line
@@
 	10400 4500 10500 4600
 Entry Wire Line
-	10400 4600 10500 4700
-Entry Wire Line
 	10400 5350 10500 5450
 Entry Wire Line
@@
 	10400 5950 10500 6050
 Entry Wire Line
-	10400 6050 10500 6150
-Entry Wire Line
-	7800 6050 7900 6150
-Entry Wire Line
 	7800 5950 7900 6050
 Entry Wire Line
@@
 	7800 4500 7900 4600
 Entry Wire Line
-	7800 4600 7900 4700
-Entry Wire Line
 	5200 3900 5300 4000
 Entry Wire Line
@@
 	5200 4500 5300 4600
 Entry Wire Line
-	5200 4600 5300 4700
-Entry Wire Line
 	5200 5350 5300 5450
 Entry Wire Line
@@
 	5200 5950 5300 6050
 Entry Wire Line
-	5200 6050 5300 6150
-Entry Wire Line
 	7800 2450 7900 2550
 Entry Wire Line
@@
 	7800 3050 7900 3150
 Entry Wire Line
-	7800 3150 7900 3250
-Entry Wire Line
 	5200 2450 5300 2550
 Entry Wire Line
@@
 	5200 3050 5300 3150
 Entry Wire Line
-	5200 3150 5300 3250
-Entry Wire Line
 	5200 950  5300 1050
 Entry Wire Line
@@
 	5200 1550 5300 1650
 Entry Wire Line
-	5200 1650 5300 1750
-Entry Wire Line
 	7800 950  7900 1050
 Entry Wire Line
@@
 Entry Wire Line
 	7800 1550 7900 1650
-Entry Wire Line
-	7800 1650 7900 1750
 Wire Wire Line
 	7150 3250 7800 3250
@@
 Text Label 2800 3950 2    50   ~ 0
 G-2
-Text Label 2800 4050 2    50   ~ 0
-DP-2
 Text Label 2800 6100 2    50   ~ 0
 D-3
@@
 Text Label 2800 6400 2    50   ~ 0
 G-3
-Text Label 2800 6500 2    50   ~ 0
-DP-3
 Text Label 5200 1350 2    50   ~ 0
 E-3
@@
 Text Label 5200 1550 2    50   ~ 0
 G-3
-Text Label 5200 1650 2    50   ~ 0
-DP-3
 Text Label 7800 950  2    50   ~ 0
 A-1
@@
 Text Label 7800 1550 2    50   ~ 0
 G-1
-Text Label 7800 1650 2    50   ~ 0
-DP-1
 Text Label 10400 950  2    50   ~ 0
 A-1
@@
 Text Label 10400 1550 2    50   ~ 0
 G-1
-Text Label 10400 1650 2    50   ~ 0
-DP-1
 Text Label 5200 2850 2    50   ~ 0
 E-1
@@
 Text Label 5200 5950 2    50   ~ 0
 G-3
-Text Label 5200 3150 2    50   ~ 0
-DP-1
-Text Label 5200 4600 2    50   ~ 0
-DP-2
-Text Label 5200 6050 2    50   ~ 0
-DP-3
-Text Label 7800 3150 2    50   ~ 0
-DP-3
-Text Label 7800 4600 2    50   ~ 0
-DP-2
-Text Label 7800 6050 2    50   ~ 0
-DP-3
 Text Label 7800 2450 2    50   ~ 0
 A-3
@@
 Text Label 10400 5950 2    50   ~ 0
 G-3
-Text Label 10400 3150 2    50   ~ 0
-DP-3
-Text Label 10400 4600 2    50   ~ 0
-DP-1
-Text Label 10400 6050 2    50   ~ 0
-DP-3
 Text Label 3000 950  0    50   ~ 0
 A-1
@@
 Text Label 3000 1550 0    50   ~ 0
 G-1
-Text Label 3000 1650 0    50   ~ 0
-DP-1
 Text Label 5400 950  0    50   ~ 0
 A-2
@@
 Text Label 5400 1550 0    50   ~ 0
 G-2
-Text Label 5400 1650 0    50   ~ 0
-DP-2
 Text Label 8000 950  0    50   ~ 0
 A-2
@@
 Text Label 8000 1550 0    50   ~ 0
 G-2
-Text Label 8000 1650 0    50   ~ 0
-DP-2
 Text Label 3000 1750 0    50   ~ 0
-EN2-6
+EN1-6
 Text Label 3000 3250 0    50   ~ 0
 EN1-1
@@
 EN3-4
 Text Label 8000 6150 0    50   ~ 0
-EN1-6
+EN2-6
 Text Label 3000 2450 0    50   ~ 0
 A-1
@@
 Text Label 5400 5950 0    50   ~ 0
 G-2
-Text Label 5400 3150 0    50   ~ 0
-DP-2
-Text Label 5400 4600 0    50   ~ 0
-DP-3
-Text Label 5400 6050 0    50   ~ 0
-DP-2
 Text Label 8000 2450 0    50   ~ 0
 A-2
@@
 Text Label 8000 5950 0    50   ~ 0
 G-2
-Text Label 8000 3150 0    50   ~ 0
-DP-2
-Text Label 8000 4600 0    50   ~ 0
-DP-3
-Text Label 8000 6050 0    50   ~ 0
-DP-2
 Wire Wire Line
 	1650 1550 1400 1550
@@
 DSKY-DSP-LCD:  LCD Decode Logic\nCopyright 2021, William Glasford
 NoConn ~ 1650 4400
-NoConn ~ 3400 3300
 NoConn ~ 1650 6850
 Text HLabel 1650 1000 0    50   Input ~ 0
@@
 Text HLabel 1650 5900 0    50   Input ~ 0
 MODE3
+NoConn ~ 9850 3150
+NoConn ~ 8650 3150
+NoConn ~ 8650 4600
+NoConn ~ 9850 4600
+NoConn ~ 9850 6050
+NoConn ~ 8650 6050
+NoConn ~ 7150 6050
+NoConn ~ 5950 6050
+NoConn ~ 5950 4600
+NoConn ~ 7150 4600
+NoConn ~ 7150 3150
+NoConn ~ 5950 3150
+NoConn ~ 4700 3150
+NoConn ~ 4700 4600
+NoConn ~ 4700 6050
+NoConn ~ 2450 6500
+NoConn ~ 2450 4050
+NoConn ~ 9850 1650
+NoConn ~ 8650 1650
+NoConn ~ 7150 1650
+NoConn ~ 5950 1650
+NoConn ~ 4700 1650
+NoConn ~ 3500 1650
 Wire Bus Line
 	950  7050 950  7600

Commit message: DSKY Redesign
Parts:
- removed U53, U54, U55: ICM7228C, symbol Driver_LED:ICM7228C
Connections:
- net labels added: BAH1, BAH2, BAH3, BAH4, BAH5, BAH6, BAH7, BAH[1..7], BAL1, BAL2, BAL3, BAL4, BAL5, BAL6, BAL7, BAL[1..7], BBH1, BBH2, BBH3, BBH4, BBH5, BBH6, BBH7, BBH[1..7], BBL1, BBL2, BBL3, BBL4, BBL5, BBL6, BBL7, BBL[1..7], DDA1, DDA11, DDA12, DDA13, DDA14, DDA15, DDA16, DDA2, DDA3, DDA5, DDA6, DDA[1..16], DDB1, DDB11, DDB12, DDB13, DDB14, DDB15, DDB2, DDB3, DDB4, DDB5, DDB[1..15], SGN1, SGN2, SGN3, SGN4, SGN5, SGN6, SGN[1..6]
- net labels removed: A-1, A-2, A-3, B-1, B-2, B-3, C-1, C-2, C-3, D-1, D-2, D-3, DA11, DA12, DA13, DA1[1..3], DA21, DA22, DA23, DA2[1..3], DA31, DA32, DA33, DA3[1..3], DP-1, E-1, E-2, E-3, EN1-1, EN1-2, EN1-3, EN1-4, EN1-5, EN1-6, EN1-7, EN1-8, EN2-1, EN2-2, EN2-3, EN2-4, EN2-5, EN2-6, EN2-7, EN2-8, EN3-1, EN3-2, EN3-3, EN3-4, EN3-5, EN3-6, EN3-7, EN3-8, F-1, F-2, F-3, G-1, G-2, G-3, GND, ID10, ID11, ID12, ID13, ID14, ID1[0..4], ID20, ID21, ID22, ID23, ID2[0..3], ID30, ID31, ID32, ID33, ID3[0..3], MODE1, MODE2, MODE3, WRITE1, WRITE2, WRITE3
- wire segments 263 -> 201
- no-connect marks 25 -> 39
Other:
- note added: "DSKY-DSP-LCD: 7-segment LCDs\nCopyright 2021, William Glasford"
- note removed: "DSKY-DSP-LCD: LCD Decode Logic\nCopyright 2021, William Glasford"
- note removed: "Decoder1"
- note removed: "Decoder2"
- note removed: "Decoder3"
- moved on the sheet: DISP1, DISP10, DISP11, DISP12, DISP2, DISP3, DISP4, DISP5, DISP6, DISP7, DISP8, DISP9
