File: schematics/DSKY/DSKY-KBD-TEST.sch (KiCad schematic (older format))
At the start: 61 parts, among them J203 Conn_02x08, J204 Conn_02x10, J300 RPI_Connector, Q17 2N3904, Q18 2N3904, Q19 2N3904, Q20 2N3904, Q21 2N3904, Q22 2N3904, Q23 2N3904, Q24 2N3904, Q25 2N3904, Q26 2N3904, Q27 2N3904, Q28 2N3904, Q29 2N3904, Q30 2N3904, Q31 2N3904, Q32 2N3904, Q33 2N3904, Q34 2N3904, Q35 2N3904, U80 74HC245

Commit message: Minor DSKY tweaks.
Parts:
- renumbered J204 to J?, J203 to J?, J300 to J?, Q17 to Q?, Q18 to Q?, Q19 to Q?, Q20 to Q?, Q21 to Q?, Q22 to Q?, Q25 to Q?, Q26 to Q?, Q24 to Q?, Q23 to Q?, Q27 to Q?, Q28 to Q?, Q29 to Q?, Q30 to Q?, Q31 to Q?, Q32 to Q?, Q33 to Q?, Q34 to Q?, Q35 to Q?, R52 to R?, R71 to R?, R53 to R?, R72 to R?, R54 to R?, R73 to R?, R55 to R?, R74 to R?, R56 to R?, R75 to R?, R57 to R?, R76 to R?, R60 to R?, R79 to R?, R61 to R?, R80 to R?, R59 to R?, R78 to R?, R58 to R?, R77 to R?, R62 to R?, R81 to R?, R63 to R?, R82 to R?, R64 to R?, R83 to R?, R65 to R?, R84 to R?, R66 to R?, R85 to R?, R67 to R?, R86 to R?, R68 to R?, R87 to R?, R69 to R?, R88 to R?, R70 to R?, R89 to R?, U80 to U?
Connections:
- net GND: no longer Q?.1 (E), Q?.1 (E), Q?.1 (E), Q?.1 (E), Q?.1 (E)
Other:
- note added: "DSKY-KBD-TEST: Raspberry PI I/F\nCopyright 2021, William Glasford"
- note removed: "DSKY-TEST: Raspberry PI I/F\nCopyright 2021, William Glasford"
