File: schematics/DSKY/DSKY.sch (KiCad schematic (older format))
At the start: 0 parts

Commit message: DSKY Redesign
Changed lines of the file:
@@
 $Descr A 11000 8500
 encoding utf-8
-Sheet 1 12
+Sheet 1 15
 Title ""
 Date ""
@@
 $EndDescr
 Entry Wire Line
-	7250 3400 7350 3500
-Wire Wire Line
-	6600 3400 7250 3400
-Entry Wire Line
 	7350 3550 7450 3450
 Wire Wire Line
@@
 CLK2
 Wire Wire Line
-	3550 3400 4100 3400
-Entry Wire Line
-	4100 3400 4200 3500
+	3550 3200 4100 3200
+Entry Wire Line
+	4100 3200 4200 3300
 Text Label 4100 3400 2    50   ~ 0
 INDC
@@
 CLK1
 Wire Wire Line
-	6600 3600 7250 3600
-Wire Wire Line
-	6600 3700 7250 3700
-Entry Wire Line
-	7250 3600 7350 3700
-Entry Wire Line
-	7250 3700 7350 3800
+	6600 3400 7250 3400
+Wire Wire Line
+	6600 3500 7250 3500
+Entry Wire Line
+	7250 3400 7350 3500
+Entry Wire Line
+	7250 3500 7350 3600
 Text Label 7250 3600 2    50   ~ 0
 KB_STR
@@
 	4200 5500 7350 5500
 Wire Wire Line
-	6600 3800 7250 3800
-Entry Wire Line
-	7250 3800 7350 3900
+	6600 3600 7250 3600
+Entry Wire Line
+	7250 3600 7350 3700
 Text Label 7250 3800 2    50   ~ 0
 INDC
-Entry Wire Line
-	4100 3300 4200 3400
 Text Label 4100 3200 2    50   ~ 0
 STBY
-Entry Wire Line
-	4200 3300 4100 3200
 Entry Wire Line
 	4200 3200 4100 3100
@@
 Wire Wire Line
 	3550 3100 4100 3100
-Wire Wire Line
-	3550 3200 4100 3200
-Wire Wire Line
-	3550 3300 4100 3300
-$Sheet
-S 2400 2900 1150 2400
-U 60F98A64
-F0 "DSKY-DSP" 50
-F1 "DSKY-DSP.sch" 50
-F2 "DSKYRST" I R 3550 3000 50
-F3 "CLK2" I R 3550 3100 50
-F4 "CH[1..15]" I R 3550 5100 50
-F5 "STBY" I R 3550 3200 50
-F6 "PARALM" I R 3550 3500 50
-F7 "DISP" I R 3550 3300 50
-F8 "INDC" I R 3550 3400 50
-F9 "SGN_CLK2" I R 3550 3700 50
-F10 "CLK3" I R 3550 3600 50
-$EndSheet
 $Sheet
 S 5600 3050 1000 2100
@@
 F11 "INDC" O R 6600 3800 50
 F12 "RPRO" O R 6600 4100 50
-F13 "SGN_CLK2" O R 6600 4300 50
-F14 "CLK3" O R 6600 4200 50
-$EndSheet
-Wire Wire Line
-	6600 3900 7250 3900
-Entry Wire Line
-	7250 3900 7350 4000
+F13 "CLK3" O R 6600 4200 50
+$EndSheet
+Wire Wire Line
+	6600 3700 7250 3700
+Entry Wire Line
+	7250 3700 7350 3800
 Text Label 7250 3900 2    50   ~ 0
 KBD1
 Wire Wire Line
-	6600 4000 7250 4000
-Entry Wire Line
-	7250 4000 7350 4100
+	6600 3800 7250 3800
+Entry Wire Line
+	7250 3800 7350 3900
 Text Label 7250 4000 2    50   ~ 0
 PARALM
@@
 Text Label 7450 3550 0    50   ~ 0
 KB_STR
-Wire Wire Line
-	6600 3500 7250 3500
-Entry Wire Line
-	7250 3500 7350 3600
 Text Label 7250 3500 2    50   ~ 0
 STBY
@@
 	8100 3250 7450 3250
 Entry Wire Line
-	4200 3600 4100 3500
+	4200 3400 4100 3300
 Text Label 4100 3500 2    50   ~ 0
 PARALM
 Wire Wire Line
-	3550 3500 4100 3500
+	3550 3300 4100 3300
 Wire Bus Line
 	8100 5050 7950 5050
@@
 DSKY Sub-System\nCopyright 2021, William Glasford
 Wire Wire Line
-	6600 4100 7250 4100
-Entry Wire Line
-	7250 4100 7350 4200
-Entry Wire Line
-	4200 3700 4100 3600
-Wire Wire Line
-	3550 3600 4100 3600
-Wire Wire Line
-	6600 4200 7250 4200
-Entry Wire Line
-	7250 4200 7350 4300
+	6600 3900 7250 3900
+Entry Wire Line
+	7250 3900 7350 4000
+Entry Wire Line
+	4200 3500 4100 3400
+Wire Wire Line
+	3550 3400 4100 3400
+Wire Wire Line
+	6600 4000 7250 4000
+Entry Wire Line
+	7250 4000 7350 4100
 Text Label 7250 4100 2    50   ~ 0
 RPRO
@@
 	8100 3750 7450 3750
 Wire Wire Line
-	6600 4300 7250 4300
-Entry Wire Line
-	7250 4300 7350 4400
-Text Label 7250 4300 2    50   ~ 0
-SGN_CLK2
-Entry Wire Line
-	4200 3800 4100 3700
-Text Label 4100 3700 2    50   ~ 0
-SGN_CLK2
-Wire Wire Line
-	3550 3700 4100 3700
-Text Label 7250 4200 2    50   ~ 0
-CLK3
-Text Label 4100 3600 2    50   ~ 0
-CLK3
+	6600 4100 7250 4100
+Entry Wire Line
+	7250 4100 7350 4200
+Entry Wire Line
+	4200 3600 4100 3500
+Wire Wire Line
+	3550 3500 4100 3500
 $Sheet
 S 3850 6050 1500 950
@@
 F1 "DSKY-TEST.sch" 50
 $EndSheet
-Wire Bus Line
-	4200 2750 4200 3850
-Wire Bus Line
-	7350 2750 7350 4450
+$Sheet
+S 2400 2900 1150 2400
+U 60F98A64
+F0 "DSKY-DSP" 50
+F1 "DSKY-DSP.sch" 50
+F2 "DSKYRST" I R 3550 3000 50
+F3 "CLK2" I R 3550 3100 50
+F4 "CH[1..15]" I R 3550 5100 50
+F5 "STBY" I R 3550 3200 50
+F6 "PARALM" I R 3550 3500 50
+F7 "DISP" I R 3550 3300 50
+F8 "INDC" I R 3550 3400 50
+F9 "CLK3" I R 3550 3600 50
+$EndSheet
+Wire Wire Line
+	6600 4200 7250 4200
+Entry Wire Line
+	7250 4200 7350 4300
+Text Label 7250 4200 2    50   ~ 0
+CLK3
+Entry Wire Line
+	4200 3700 4100 3600
+Text Label 4100 3600 2    50   ~ 0
+CLK3
+Wire Wire Line
+	3550 3600 4100 3600
+Wire Bus Line
+	4200 2750 4200 3750
+Wire Bus Line
+	7350 2750 7350 4350
 $EndSCHEMATC

Commit message: Minor DSKY tweaks.
Changed lines of the file:
@@
 F12 "RPRO" O R 6600 4100 50
 F13 "CLK3" O R 6600 4200 50
+F14 "SGNRST" O R 6600 4300 50
 $EndSheet
 Wire Wire Line
@@
 	3550 3500 4100 3500
 $Sheet
-S 3850 6050 1500 950
-U 62ECFB9F
-F0 "DSKY-TEST" 50
-F1 "DSKY-TEST.sch" 50
-$EndSheet
-$Sheet
 S 2400 2900 1150 2400
 U 60F98A64
@@
 F8 "INDC" I R 3550 3400 50
 F9 "CLK3" I R 3550 3600 50
+F10 "SGNRST" I R 3550 3700 50
 $EndSheet
 Wire Wire Line
@@
 Wire Wire Line
 	3550 3600 4100 3600
+$Sheet
+S 4400 5950 1200 900
+U 6A27E71F
+F0 "DSKY-TEST" 50
+F1 "DSKY-TEST.sch" 50
+$EndSheet
+Wire Wire Line
+	6600 4300 7250 4300
+Entry Wire Line
+	7250 4300 7350 4400
+Text Label 7250 4300 2    50   ~ 0
+SGNRST
+Entry Wire Line
+	4200 3800 4100 3700
+Text Label 4100 3700 2    50   ~ 0
+SGNRST
+Wire Wire Line
+	3550 3700 4100 3700
 Wire Bus Line
-	4200 2750 4200 3750
+	4200 2750 4200 3900
 Wire Bus Line
-	7350 2750 7350 4350
+	7350 2750 7350 4500
 $EndSCHEMATC
