File: schematics/DSKY/DSKY_DSP_SGN.sch (KiCad schematic (older format))
At the start: 16 parts, among them U18 74LS00, U19 74LS04, U42 74LS04, U46 74LS86, U60 74LS112, U61 74LS112, U62 74LS112, U63 74LS112, U64 74LS02, U79 74LS04

Commit message: Minor DSKY tweaks.
Connections:
- net DSKYRST renamed SGNRST
Changed lines of the file:
@@
 $Descr A 8500 11000 portrait
 encoding utf-8
-Sheet 10 15
+Sheet 9 15
 Title ""
 Date ""
@@
 Connection ~ 2750 8550
 Text HLabel 2600 8550 0    50   Input ~ 0
-DSKYRST
+SGNRST
 Wire Bus Line
 	750  1050 750  1300
