File: schematics/DSKY/DSKY_DSP_CTL.sch (KiCad schematic (older format))
At the start: 23 parts, among them U17 74LS04, U38 74LS74, U40 LM555, U41 LM555, U48 74LS00, U54 74LS08, U68 74LS112, U69 74LS161, U70 74LS154, U72 74LS02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

Commit message: New Display Logic Using ICM7128s
Parts:
- removed R13: 1K, symbol Device:R_US
- removed unit 3 of U54
- removed U75: 74LS32, symbol 74xx:74LS32
- removed U77: 74LS86, symbol 74xx:74LS86
- added unit 2 of U17
- added unit 2 of U38
- added unit 2 of U48
- added unit 3 of U48
- added unit 4 of U54
- added unit 2 of U72
- added unit 3 of U72
- added unit 4 of U72
- added unit 2 of U73
- added unit 3 of U73
- added U75: 74LS74, symbol 74xx:74LS74
- added U77: 74LS30, symbol 74xx:74LS30
- added U78: 74LS27, symbol 74xx:74LS27
- added U79: 74LS10, symbol 74xx:74LS10
- added U80: 74LS112, symbol 74xx:74LS112
- added U81: 74LS08, symbol 74xx:74LS08
- C5: value 1uF -> .001uF
Connections:
- net labels added: D0, D1, D2, D3, D4
- wire segments 188 -> 256
- no-connect marks 4 -> 5
Other:
- note added: "5th Digit:\nDelay one pulse \noff TC (1111)"
- note added: "Mode needs to be a \nsingle pulse before \nthe write pulses to\ncause a read of the \ncontrol data."
- note added: "Mode/\nData"
- note added: "Note: The NOR gates\ncould be replaced by\na NOT and OR gate.\nThis was done to\nreduce the chip count."
- note added: "Start State:\n11110"
- note added: "State: 10000\nStop counting"
- note added: "State: 11111"
- note added: "Write"
- note removed: "Cycle Display"
- note removed: "Rotate through the \nbanks of registers,\nenabling one at a time."
- moved on the sheet: C4, C6, C7, R12, R4, R5, RV1, U17A, U38A, U67, U68A, U68B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

Commit message: Modified to use fourth display decoder chip.
Parts:
- added unit 6 of U17
Connections:
- net labels added: DE[0..15]
- net labels removed: DE[1..11]
- wire segments 256 -> 258
Other:
- moved on the sheet: U17E, U70
