File: schematics/DSKY/DSKY_DSP_REG.sch (KiCad schematic (older format))
At the start: 13 parts, among them U52 74LS244, U53 74LS244, U56 74LS374, U57 74LS374, U58 74LS374, U59 74LS374, U60 74LS374, U61 74LS374, U62 74LS374, U63 74LS374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

Commit message: Modified to use fourth display decoder chip.
Connections:
- net DE1: now also U61.1 (OE); no longer U66.1 (OE)
- net DE2: now also U62.1 (OE); no longer U65.1 (OE)
- net DE3: now also U63.1 (OE); no longer U64.1 (OE)
- net DE4: now also U64.1 (OE); no longer U63.1 (OE)
- net DE5: now also U65.1 (OE); no longer U62.1 (OE)
- net DE6: now also U66.1 (OE); no longer U61.1 (OE)
- net DE10 renamed DE13
- net DE11 renamed DE12
- net DE7 renamed DE0
- net DE8 renamed DE15
- net DE9 renamed DE14
- net RWD1 renamed nRWD1
- net RWD10 renamed nRWD10
- net RWD11 renamed nRWD11
- net RWD2 renamed nRWD2
- net RWD3 renamed nRWD3
- net RWD4 renamed nRWD4
- net RWD5 renamed nRWD5
- net RWD6 renamed nRWD6
- net RWD7 renamed nRWD7
- net RWD8 renamed nRWD8
- net RWD9 renamed nRWD9
Other:
- note added: "Note: The DE pulses are \nreversed because the\ndata needs to go to the\ndriver chips in reverse."
Changed lines of the file:
@@
 $Descr A 8500 11000 portrait
 encoding utf-8
-Sheet 9 13
+Sheet 9 14
 Title ""
 Date ""
@@
 DSKY-DSP-REG:  Display Registers\nCopyright 2021, William Glasford
 $Comp
-L 74xx:74LS374 U56
-U 1 1 65CA45F9
-P 1550 1600
-F 0 "U56" H 1800 2400 50  0000 C CNN
-F 1 "74LS374" H 1800 2300 50  0000 C CNN
-F 2 "" H 1550 1600 50  0001 C CNN
-F 3 "http://www.ti.com/lit/gpn/sn74LS374" H 1550 1600 50  0001 C CNN
-	1    1550 1600
-	1    0    0    -1
-$EndComp
-$Comp
 L 74xx:74LS374 U59
 U 1 1 65CA5D19
@@
 BCD[1..8]
 Text HLabel 1550 2800 0    50   Input ~ 0
-DE[1..11]
+DE[0..15]
 Wire Bus Line
 	2400 650  2550 650
@@
 Wire Bus Line
 	1650 2800 1650 2900
-Text HLabel 2200 2750 0    50   Input ~ 0
-RWD[1..11]
 Entry Wire Line
 	4300 1200 4400 1100
@@
 	800  1800 1050 1800
 Wire Bus Line
-	2300 2750 2200 2750
-Wire Bus Line
-	2300 2650 2300 2750
-Wire Bus Line
 	2400 550  2400 650
 Connection ~ 2400 650
@@
 Entry Wire Line
 	1050 2800 1150 2900
-Connection ~ 2300 2650
 Connection ~ 1650 2900
-Wire Wire Line
-	1050 2100 1050 2800
 Entry Wire Line
 	2850 5200 2950 5300
@@
 R3D4\n\n\nR3D5
 Text Label 850  2550 1    50   ~ 0
-RWD11
+nRWD11
 Text Label 2650 2550 1    50   ~ 0
-RWD8
+nRWD8
 Text Label 850  4950 1    50   ~ 0
-RWD10
+nRWD10
 Text Label 850  7300 1    50   ~ 0
-RWD9
+nRWD9
 Text Label 2650 4950 1    50   ~ 0
-RWD7
+nRWD7
 Text Label 2650 7300 1    50   ~ 0
-RWD6
+nRWD6
 Text Label 4450 2550 1    50   ~ 0
-RWD5
+nRWD5
 Text Label 4450 4950 1    50   ~ 0
-RWD4
+nRWD4
 Text Label 4450 7300 1    50   ~ 0
-RWD3
+nRWD3
 Text Label 6250 2550 1    50   ~ 0
-RWD2
+nRWD2
 Text Label 6250 4950 1    50   ~ 0
-RWD1
+nRWD1
 Text Label 4650 2800 2    50   ~ 0
-DE5
+DE2
 Text Label 4650 5200 2    50   ~ 0
+DE3
+Text Label 4650 7550 2    50   ~ 0
 DE4
-Text Label 4650 7550 2    50   ~ 0
-DE3
 Wire Bus Line
 	600  2900 600  5300
@@
 Connection ~ 2500 7750
 Text Label 6450 2800 2    50   ~ 0
-DE2
+DE5
 Text Label 6450 5200 2    50   ~ 0
+DE6
+Text Label 2850 2800 2    50   ~ 0
+DE15
+Text Label 2850 5200 2    50   ~ 0
+DE0
+Text Label 2850 7550 2    50   ~ 0
 DE1
-Text Label 2850 2800 2    50   ~ 0
-DE8
-Text Label 2850 5200 2    50   ~ 0
-DE7
-Text Label 2850 7550 2    50   ~ 0
-DE6
 Text Label 1050 2800 2    50   ~ 0
-DE11
+DE12
 Text Label 900  8400 0    50   ~ 0
 BCD1
@@
 	1050 7550 1150 7650
 Text Label 1050 7550 2    50   ~ 0
-DE9
+DE14
 Wire Wire Line
 	1050 4500 1050 5200
@@
 	1050 5200 1150 5300
 Text Label 1050 5200 2    50   ~ 0
-DE10
+DE13
+Wire Wire Line
+	1050 2100 1050 2800
+Wire Bus Line
+	2300 2650 2300 2550
+Wire Bus Line
+	2300 2550 2200 2550
+Text HLabel 2200 2550 0    50   Input ~ 0
+nRWD[1..11]
+$Comp
+L 74xx:74LS374 U56
+U 1 1 65CA45F9
+P 1550 1600
+F 0 "U56" H 1800 2400 50  0000 C CNN
+F 1 "74LS374" H 1800 2300 50  0000 C CNN
+F 2 "" H 1550 1600 50  0001 C CNN
+F 3 "http://www.ti.com/lit/gpn/sn74LS374" H 1550 1600 50  0001 C CNN
+	1    1550 1600
+	1    0    0    -1
+$EndComp
+Connection ~ 2300 2650
+Text Notes 6350 6200 0    50   ~ 0
+Note: The DE pulses are \nreversed because the\ndata needs to go to the\ndriver chips in reverse.
 Wire Bus Line
 	600  2900 1650 2900
